Commit message: sync pika gripper ee frame with franka hand frame; add umi data collection; partially fix docker; update act && fixed sim

File: assets/franka_fr3/fr3_pika_gripper_ati.urdf (robot description, URDF)
Before this commit: robot fr3, 17 links, 16 joints
Joints:
- joint ati_pika_joint: origin xyz=0.0 0.0 0.0 rpy=0.0 0.0 0 -> xyz=0.0 0.0 0.0 rpy=-0.739815 0.0 0.0 
- joint fr3_hand_tcp_joint: origin xyz=0.185 0 0 rpy=0 0 0 -> xyz=0.185 0 0 rpy=3.1415926 -1.5707963 0

Commit message: fr3 bp umi infer ok

File: assets/franka_fr3/fr3_pika_gripper_ati.urdf (robot description, URDF)
Before this commit: robot fr3, 17 links, 16 joints
Joints:
- joint fr3_joint2: limit lower=-1.7837 upper=1.7837 effort=87.0 velocity=2.62 -> lower=-1.76 upper=1.76 effort=87.0 velocity=2.62
