Commit message: support single zmq gripper and camera and original g1 ik and tested chunk action for unitree

File: assets/unitree_g1/g1_29dof_with_hand.urdf (robot description, URDF)
Before this commit: robot g1_29dof_with_hand, 55 links, 54 joints
Links:
- added link left_tcp
- added link right_tcp
- link head_link: geometry collision mesh filename=/workspace/assets/unitree_g1/meshes/head_link.STL; visual mesh filename=/workspace/assets/unitree_g1/meshes/head_link.STL
- link left_ankle_pitch_link: geometry collision mesh filename=/workspace/assets/unitree_g1/meshes/left_ankle_pitch_link.S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; visual mesh filename=/workspace/assets/unitree_g1/meshes/left_ankle_pitch_link.S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
- link left_ankle_roll_link: geometry collision sphere radius=0.005; collision sphere radius=0.005
- link left_elbow_link: geometry collision mesh filename=/workspace/assets/unitree_g1/meshes/left_elbow_link.STL; visual mesh filename=/workspace/assets/unitree_g1/meshes/left_elbow_link.STL
- link left_hand_index_0_link: geometry collision mesh filename=/workspace/assets/unitree_g1/meshes/left_hand_index_0_link.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; visual mesh filename=/workspace/assets/unitree_g1/meshes/left_hand_index_0_link.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
- link left_hand_index_1_link: geometry collision mesh filename=/workspace/assets/unitree_g1/meshes/left_hand_index_1_link.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; visual mesh filename=/workspace/assets/unitree_g1/meshes/left_hand_index_1_link.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
- link left_hand_middle_0_link: geometry collision mesh filename=/workspace/assets/unitree_g1/meshes/left_hand_middle_0_link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; visual mesh filename=/workspace/assets/unitree_g1/meshes/left_hand_middle_0_link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
- link left_hand_middle_1_link: geometry collision mesh filename=/workspace/assets/unitree_g1/meshes/left_hand_middle_1_link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; visual mesh filename=/workspace/assets/unitree_g1/meshes/left_hand_middle_1_link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
- link left_hand_palm_link: geometry collision mesh filename=/workspace/assets/unitree_g1/meshes/left_hand_palm_link.STL; visual mesh filename=/workspace/assets/unitree_g1/meshes/left_hand_palm_link.STL
- link left_hand_thumb_0_link: geometry collision mesh filename=/workspace/assets/unitree_g1/meshes/left_hand_thumb_0_link.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; visual mesh filename=/workspace/assets/unitree_g1/meshes/left_hand_thumb_0_link.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
- link left_hand_thumb_1_link: geometry collision box size=0.02 0.03 0.02; visual mesh filename=/workspace/assets/unitree_g1/meshes/left_hand_thumb_1_link.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
- link left_hand_thumb_2_link: geometry collision mesh filename=/workspace/assets/unitree_g1/meshes/left_hand_thumb_2_link.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; visual mesh filename=/workspace/assets/unitree_g1/meshes/left_hand_thumb_2_link.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
- link left_hip_pitch_link: geometry collision mesh filename=/workspace/assets/unitree_g1/meshes/left_hip_pitch_link.STL; visual mesh filename=/workspace/assets/unitree_g1/meshes/left_hip_pitch_link.STL
- link left_hip_roll_link: geometry collision mesh filename=/workspace/assets/unitree_g1/meshes/left_hip_roll_link.STL; visual mesh filename=/workspace/assets/unitree_g1/meshes/left_hip_roll_link.STL
- link left_hip_yaw_link: geometry collision mesh filename=/workspace/assets/unitree_g1/meshes/left_hip_yaw_link.STL; visual mesh filename=/workspace/assets/unitree_g1/meshes/left_hip_yaw_link.STL
- link left_knee_link: geometry collision mesh filename=/workspace/assets/unitree_g1/meshes/left_knee_link.STL; visual mesh filename=/workspace/assets/unitree_g1/meshes/left_knee_link.STL
- link left_shoulder_pitch_link: geometry collision cylinder length=0.05 radius=0.03; visual mesh filename=/workspace/assets/unitree_g1/meshes/left_shoulder_pitch_lin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
- link left_shoulder_roll_link: geometry collision cylinder length=0.03 radius=0.03; visual mesh filename=/workspace/assets/unitree_g1/meshes/left_shoulder_roll_link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
- link left_shoulder_yaw_link: geometry collision mesh filename=/workspace/assets/unitree_g1/meshes/left_shoulder_yaw_link.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; visual mesh filename=/workspace/assets/unitree_g1/meshes/left_shoulder_yaw_link.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
- link left_wrist_pitch_link: geometry collision mesh filename=/workspace/assets/unitree_g1/meshes/left_wrist_pitch_link.S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; visual mesh filename=/workspace/assets/unitree_g1/meshes/left_wrist_pitch_link.S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
- link left_wrist_roll_link: geometry collision mesh filename=/workspace/assets/unitree_g1/meshes/left_wrist_roll_link.STL; visual mesh filename=/workspace/assets/unitree_g1/meshes/left_wrist_roll_link.STL
- link left_wrist_yaw_link: geometry collision mesh filename=/workspace/assets/unitree_g1/meshes/left_wrist_yaw_link.STL; visual mesh filename=/workspace/assets/unitree_g1/meshes/left_wrist_yaw_link.STL
- link logo_link: geometry collision mesh filename=/workspace/assets/unitree_g1/meshes/logo_link.STL; visual mesh filename=/workspace/assets/unitree_g1/meshes/logo_link.STL
- link pelvis: geometry visual mesh filename=/workspace/assets/unitree_g1/meshes/pelvis.STL
- link pelvis_contour_link: geometry collision mesh filename=/workspace/assets/unitree_g1/meshes/pelvis_contour_link.STL; visual mesh filename=/workspace/assets/unitree_g1/meshes/pelvis_contour_link.STL
- link right_ankle_pitch_link: geometry collision mesh filename=/workspace/assets/unitree_g1/meshes/right_ankle_pitch_link.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; visual mesh filename=/workspace/assets/unitree_g1/meshes/right_ankle_pitch_link.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
- link right_ankle_roll_link: geometry collision sphere radius=0.005; collision sphere radius=0.005
- link right_elbow_link: geometry collision mesh filename=/workspace/assets/unitree_g1/meshes/right_elbow_link.STL; visual mesh filename=/workspace/assets/unitree_g1/meshes/right_elbow_link.STL
- link right_hand_index_0_link: geometry collision mesh filename=/workspace/assets/unitree_g1/meshes/right_hand_index_0_link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; visual mesh filename=/workspace/assets/unitree_g1/meshes/right_hand_index_0_link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
- link right_hand_index_1_link: geometry collision mesh filename=/workspace/assets/unitree_g1/meshes/right_hand_index_1_link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; visual mesh filename=/workspace/assets/unitree_g1/meshes/right_hand_index_1_link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
- link right_hand_middle_0_link: geometry collision mesh filename=/workspace/assets/unitree_g1/meshes/right_hand_middle_0_lin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; visual mesh filename=/workspace/assets/unitree_g1/meshes/right_hand_middle_0_lin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
- link right_hand_middle_1_link: geometry collision mesh filename=/workspace/assets/unitree_g1/meshes/right_hand_middle_1_lin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; visual mesh filename=/workspace/assets/unitree_g1/meshes/right_hand_middle_1_lin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
- link right_hand_palm_link: geometry collision mesh filename=/workspace/assets/unitree_g1/meshes/right_hand_palm_link.STL; visual mesh filename=/workspace/assets/unitree_g1/meshes/right_hand_palm_link.STL
- link right_hand_thumb_0_link: geometry collision mesh filename=/workspace/assets/unitree_g1/meshes/right_hand_thumb_0_link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; visual mesh filename=/workspace/assets/unitree_g1/meshes/right_hand_thumb_0_link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
- link right_hand_thumb_1_link: geometry collision box size=0.02 0.03 0.02; visual mesh filename=/workspace/assets/unitree_g1/meshes/right_hand_thumb_1_link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
- link right_hand_thumb_2_link: geometry collision mesh filename=/workspace/assets/unitree_g1/meshes/right_hand_thumb_2_link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; visual mesh filename=/workspace/assets/unitree_g1/meshes/right_hand_thumb_2_link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
- link right_hip_pitch_link: geometry collision mesh filename=/workspace/assets/unitree_g1/meshes/right_hip_pitch_link.STL; visual mesh filename=/workspace/assets/unitree_g1/meshes/right_hip_pitch_link.STL
- link right_hip_roll_link: geometry collision mesh filename=/workspace/assets/unitree_g1/meshes/right_hip_roll_link.STL; visual mesh filename=/workspace/assets/unitree_g1/meshes/right_hip_roll_link.STL
- link right_hip_yaw_link: geometry collision mesh filename=/workspace/assets/unitree_g1/meshes/right_hip_yaw_link.STL; visual mesh filename=/workspace/assets/unitree_g1/meshes/right_hip_yaw_link.STL
- link right_knee_link: geometry collision mesh filename=/workspace/assets/unitree_g1/meshes/right_knee_link.STL; visual mesh filename=/workspace/assets/unitree_g1/meshes/right_knee_link.STL
- link right_shoulder_pitch_link: geometry collision cylinder length=0.05 radius=0.03; visual mesh filename=/workspace/assets/unitree_g1/meshes/right_shoulder_pitch_li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
- link right_shoulder_roll_link: geometry collision cylinder length=0.03 radius=0.03; visual mesh filename=/workspace/assets/unitree_g1/meshes/right_shoulder_roll_lin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
- link right_shoulder_yaw_link: geometry collision mesh filename=/workspace/assets/unitree_g1/meshes/right_shoulder_yaw_link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; visual mesh filename=/workspace/assets/unitree_g1/meshes/right_shoulder_yaw_link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
- link right_wrist_pitch_link: geometry collision mesh filename=/workspace/assets/unitree_g1/meshes/right_wrist_pitch_link.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; visual mesh filename=/workspace/assets/unitree_g1/meshes/right_wrist_pitch_link.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
- link right_wrist_roll_link: geometry collision mesh filename=/workspace/assets/unitree_g1/meshes/right_wrist_roll_link.S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; visual mesh filename=/workspace/assets/unitree_g1/meshes/right_wrist_roll_link.S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
- link right_wrist_yaw_link: geometry collision mesh filename=/workspace/assets/unitree_g1/meshes/right_wrist_yaw_link.STL; visual mesh filename=/workspace/assets/unitree_g1/meshes/right_wrist_yaw_link.STL
- link torso_link: geometry collision mesh filename=/workspace/assets/unitree_g1/meshes/torso_link.STL; visual mesh filename=/workspace/assets/unitree_g1/meshes/torso_link.STL
- link waist_roll_link: geometry visual mesh filename=/workspace/assets/unitree_g1/meshes/waist_roll_link.STL
- link waist_support_link: geometry collision mesh filename=/workspace/assets/unitree_g1/meshes/waist_support_link.STL; visual mesh filename=/workspace/assets/unitree_g1/meshes/waist_support_link.STL
- link waist_yaw_link: geometry visual mesh filename=/workspace/assets/unitree_g1/meshes/waist_yaw_link.STL
Joints:
- added joint left_tcp_joint: type fixed, parent left_hand_palm_link, child left_tcp, origin xyz=0.18 0 0 rpy=0 0 0
- added joint right_tcp_joint: type fixed, parent right_hand_palm_link, child right_tcp, origin xyz=0.18 0 0 rpy=0 0 0
